File: preamp.sch (EAGLE design)
At the start: 74 parts, among them IC1 OPAMP-DUALDIP, IC2 OPAMP-DUALDIP, IC3 QUAD_OPAMPP, IC4 OPAMP-DUALDIP, IC5 OPAMP-DUALDIP, IC6 QUAD_OPAMPP, J1 Instrument Input, J2 Instrument Output, SW1 SWITCH_DPDT

Commit message: fixed schematic, started layout
Parts:
- removed C10: 6.8uF, SparkFun-Capacitors:CAPPTH1
- removed IC4, IC5: OPAMP-DUALDIP, SparkFun-AnalogIC:OPAMP-DUALDIP
- removed IC6: QUAD_OPAMPP, adafruit:QUAD_OPAMPP
- added C23, C24: 470uF, SparkFun-Passives:CAP_POLPTH1
- added C25: 47nF, preamp:CAP
- added C26: 10uF, SparkFun-Capacitors:CAP_POLPTH2
- added IC7: OPAMP-QUADTL074, Op Amps:OPAMP-QUADTL074
- added JP1: M02JST-PTH-2, SparkFun-Connectors:M02JST-PTH-2
- added R14, R45: 10k, SparkFun-Passives:RESISTORPTH-1/4W
- C1: device SparkFun-Capacitors:CAPPTH1 -> preamp:CAP; PARTNO (none) -> FK28X7R1H473K
- C11, C12, C17, C18, C4: device SparkFun-Capacitors:CAPPTH1 -> preamp:CAP; PARTNO (none) -> FK28X7R1C224K
- C13, C16, C21, C22, C5: device SparkFun-Capacitors:CAPPTH1 -> preamp:CAP; PARTNO (none) -> FK28X5R1A684K
- C14, C15, C19, C20, C8: device SparkFun-Capacitors:CAPPTH1 -> preamp:CAP
- C2, C6: device SparkFun-Capacitors:CAPPTH1 -> preamp:CAP; PARTNO (none) -> FK28X5R1A335K
- C3: value 10uF -> 6.8uF; device SparkFun-Capacitors:CAPPTH1 -> SparkFun-Capacitors:CAP_POLPTH2; PARTNO (none) -> ESH685M063AC3AA
- C7, C9: device SparkFun-Capacitors:CAPPTH1 -> SparkFun-Capacitors:CAP_POLPTH2; PARTNO (none) -> ESH685M063AC3AA
- IC1, IC2: value OPAMP-DUALDIP -> OPAMP-QUADTL074; device SparkFun-AnalogIC:OPAMP-DUALDIP -> Op Amps:OPAMP-QUADTL074; PARTNO (none) -> TL074CN
- IC3: value QUAD_OPAMPP -> OPAMP-DUALDIP; device adafruit:QUAD_OPAMPP -> SparkFun-AnalogIC:OPAMP-DUALDIP; PARTNO (none) -> TL072IP
- R1, R15: PARTNO (none) -> CF14JT1M00
- R10, R11, R12, R17, R20, R21, R27, R29, R31, R4, R40, R42, R7, R8, R9: PARTNO (none) -> CF14JT10K0
- R13, R34, R37, R5: PARTNO (none) -> CF14JT12K0
- R16: PARTNO (none) -> CF14JT6K80
- R18, R22: PARTNO (none) -> CF14JT68R0
- R19, R23: PARTNO (none) -> CF14JT4K70
- R2: PARTNO (none) -> CF14JT100K
- R24: PARTNO (none) -> CF14JT15K0
- R25: PARTNO (none) -> CF14JT2K20
- R26, R28, R30, R39: PARTNO (none) -> CF14JT22K0
- R3: PARTNO (none) -> CF14JT9K10
- R32, R33, R41, R43: device preamp:POT -> preamp:POTBOURNS; PARTNO (none) -> PTV09A-2020F-B104
- R44, R6: device preamp:POT -> preamp:POTPANA; PARTNO (none) -> EVU-E2AF25D24
Connections:
- net EQ renamed N$19
- net N$27 renamed XLR_HOT
- net N$31 renamed XLR_NEG
- removed net N$19 (its old number): IC4A.-IN, R13.2, R44.A
- new net N$46: IC7A.IN-, IC7A.OUT, SW1.C1
- new net N$48: C24.-, JP1.1, R45.1
- net BOOST: now also IC2B.IN-; no longer IC3C.-IN
- net CUT: now also IC7D.IN-; no longer IC3A.-IN
- net GND: now also C23.-, C25.2, IC1SUP.VEE, IC2SUP.VEE, IC3A.V-, IC7SUP.VEE; no longer IC1A.V-, IC2A.V-, IC4A.V-, IC5A.V-
- net N$10: now also C26.-, IC7C.OUT, R6.E, R6.S; no longer IC2A.-IN, R5.2, R6.A
- net N$11: now also IC2C.IN-, R13.2, R44.A; no longer C3.1, IC2A.OUT, R6.E, R6.S
- net N$12: now also C26.+; no longer C3.2
- net N$13: now also IC7D.OUT; no longer IC3A.OUT
- net N$15: now also IC2A.IN-; no longer IC3B.-IN
- net N$16: now also IC2A.OUT; no longer IC3B.OUT
- net N$17: now also IC2B.OUT; no longer IC3C.OUT
- net N$2: now also IC7A.IN+; no longer IC1A.+IN
- net N$20: now also C3.-, IC2C.OUT; no longer C7.1, IC4A.OUT
- net N$21: now also C3.+, IC2D.IN+; no longer C7.2, IC4B.+IN
- net N$22: now also IC2D.IN-, IC2D.OUT, IC3A.+IN; no longer IC4B.-IN, IC4B.OUT, IC5A.+IN
- net N$25: now also C7.-, IC3A.-IN, IC3A.OUT; no longer C9.1, IC5A.-IN, IC5A.OUT
- net N$26: now also C7.+; no longer C9.2
- net N$28: now also IC3B.-IN; no longer IC5B.-IN
- net N$29: now also C9.-, IC3B.OUT; no longer C10.1, IC5B.OUT
- net N$3: now also IC7C.IN-, R5.2, R6.A; no longer IC1A.-IN, IC1A.OUT, SW1.C1
- net N$30: now also C9.+; no longer C10.2
- net N$32: now also IC1A.IN-; no longer IC6A.-IN
- net N$33: now also IC1A.OUT; no longer IC6A.OUT
- net N$36: now also IC1B.IN-; no longer IC6B.-IN
- net N$37: now also IC1B.OUT; no longer IC6B.OUT
- net N$42: now also IC1C.IN-; no longer IC6D.-IN
- net N$43: now also IC1C.OUT; no longer IC6D.OUT
- net N$45: now also IC1D.IN-; no longer IC6C.-IN
- net N$5: now also IC7B.IN+; no longer IC1B.+IN
- net N$51: now also IC1D.OUT; no longer IC6C.OUT
- net N$8: now also IC7B.IN-, IC7B.OUT; no longer IC1B.-IN, IC1B.OUT
- net VCC: now also C23.+, C25.1, IC1SUP.VCC, IC2SUP.VCC, IC3A.V+, IC7SUP.VCC, JP1.2, R14.2; no longer IC1A.V+, IC2A.+IN, IC2A.V+, IC4A.V+, IC5A.V+, IC5B.+IN, R2.1, R4.1
- net VCC/2: now also C24.+, IC1A.IN+, IC1B.IN+, IC1C.IN+, IC1D.IN+, IC2A.IN+, IC2B.IN+, IC2C.IN+, IC7C.IN+, IC7D.IN+, R14.1, R2.1, R4.1, R45.2; no longer IC3A.+IN, IC3C.+IN, IC4A.+IN, IC6A.+IN, IC6B.+IN, IC6C.+IN, IC6D.+IN
Other:
- note added: "Boost Summing Amp"
- note added: "Buffer"
- note added: "Cut Summing Amp"
- note added: "EQ Buffer"
- note added: "EQ Section"
- note added: "Input Buffer"
- note added: "Input Gain"
- note added: "Output Gain"
- note added: "Output Section"
- note added: "Pad Switch"
- note added: "Power"
- note removed: "CHECK POLARITY"
- note removed: "WHERE IS POWER"
- moved on the sheet: C1, C11, C12, C13, C14, C15, C16, C17, C18, C19, C2, C20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
